File: udap-usb-a.kicad_pcb (KiCad board)
At the start: 2 copper layers, 28.5 x 14.1 mm, 24 parts, among them J201 Conn_02x04_Counter_Clockwise, P101 USB_A, U2 MIC5245-3.3YM5, U201 NUF6401MNT1, U202 STM32F042F6Px, U4 NUF2042XV6T1G

Commit message: Added ferrite bead on 5V, PC EMI -> TARGET issue mitigation
Parts:
- added FB101: Ferrite_Bead_Small, passive:R_0402, F.Cu at (93.4, 109.8)
Connections:
- P101 pad 1: +5V -> Net-(FB101-Pad2)
Routing:
- net +5V: track 25.1 -> 22.0 mm
- net Net-(FB101-Pad2): track 0.00 -> 2.17 mm
Changed lines of the file:
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@@
-(kicad_pcb (version 20171130) (host pcbnew 5.1.4)
+(kicad_pcb (version 20171130) (host pcbnew 5.1.4-e60b266~84~ubuntu18.04.1)
   (general
     (thickness 0.7)
     (drawings 29)
-    (tracks 230)
+    (tracks 233)
     (zones 0)
-    (modules 24)
-    (nets 34)
+    (modules 25)
+    (nets 35)
   )
   (page A4)
@@
     (solder_mask_min_width 0.07)
     (aux_axis_origin 0 0)
-    (visible_elements FFFFFFFF)
+    (visible_elements FFFFFF7F)
     (pcbplotparams
       (layerselection 0x011f8_ffffffff)
@@
   (net 32 "Net-(D1-Pad1)")
   (net 33 "Net-(D201-Pad1)")
+  (net 34 "Net-(FB101-Pad2)")
   (net_class Default "This is the default net class."
     (clearance 0.15)
@@
     (add_net "Net-(D201-Pad1)")
     (add_net "Net-(F1-Pad1)")
+    (add_net "Net-(FB101-Pad2)")
     (add_net "Net-(U2-Pad4)")
     (add_net "Net-(U202-Pad10)")
@@
     (add_net +3V3)
     (add_net +5V)
+  )
+  (module passive:R_0402 (layer F.Cu)
+    (at 93.4 109.8 180)
+    (descr "Resistor SMD 0402 (1005 Metric), square (rectangular) end terminal, IPC_7351 nominal, (Body size source: http://www.tortai-tech.com/upload/download/2011102023233369053.pdf), generated with kicad-footprint-generator")
+    (tags resistor)
+    (attr smd)
+    (fp_text reference FB101 (at -1.8 0) (layer F.SilkS) hide
+      (effects (font (size 0.6 0.6) (thickness 0.13)))
+    )
+    (fp_text value Ferrite_Bead_Small (at 0 0.45) (layer F.Fab) hide
+      (effects (font (size 0.2 0.2) (thickness 0.03)))
+    )
+    (fp_line (start 0 -0.3) (end 0 0.3) (layer F.SilkS) (width 0.15))
+    (fp_line (start -0.5 0.25) (end -0.5 -0.25) (layer F.Fab) (width 0.1))
+    (fp_line (start -0.5 -0.25) (end 0.5 -0.25) (layer F.Fab) (width 0.1))
+    (fp_line (start 0.5 -0.25) (end 0.5 0.25) (layer F.Fab) (width 0.1))
+    (fp_line (start 0.5 0.25) (end -0.5 0.25) (layer F.Fab) (width 0.1))
+    (fp_line (start -0.8 0.4) (end -0.8 -0.4) (layer F.CrtYd) (width 0.05))
+    (fp_line (start -0.8 -0.4) (end 0.8 -0.4) (layer F.CrtYd) (width 0.05))
+    (fp_line (start 0.8 -0.4) (end 0.8 0.4) (layer F.CrtYd) (width 0.05))
+    (fp_line (start 0.8 0.4) (end -0.8 0.4) (layer F.CrtYd) (width 0.05))
+    (fp_text user %R (at 0 0) (layer F.Fab)
+      (effects (font (size 0.2 0.2) (thickness 0.03)))
+    )
+    (pad 1 smd roundrect (at -0.4 0 180) (size 0.55 0.55) (layers F.Cu F.Paste F.Mask) (roundrect_rratio 0.25)
+      (net 3 +5V))
+    (pad 2 smd roundrect (at 0.4 0 180) (size 0.55 0.55) (layers F.Cu F.Paste F.Mask) (roundrect_rratio 0.25)
+      (net 34 "Net-(FB101-Pad2)"))
+    (model ${KISYS3DMOD}/Resistor_SMD.3dshapes/R_0402_1005Metric.step
+      (at (xyz 0 0 0))
+      (scale (xyz 1 1 1))
+      (rotate (xyz 0 0 0))
+    )
   )
   (module usb:USB_A_1001-011-01101 (layer F.Cu)
@@
     (pad "" np_thru_hole circle (at 2.3 2.1 180) (size 1.2 1.2) (drill 1.2) (layers *.Cu *.Mask))
     (pad 1 smd roundrect (at 3.56 -0.75 180) (size 2.5 1.2) (layers F.Cu F.Mask) (roundrect_rratio 0.25)
-      (net 3 +5V))
+      (net 34 "Net-(FB101-Pad2)"))
     (pad 2 smd roundrect (at 1.02 -0.75 180) (size 2.5 1.2) (layers F.Cu F.Mask) (roundrect_rratio 0.25)
       (net 4 /DM))
@@
   (segment (start 94.1 102.4) (end 94.18001 102.31999) (width 0.4) (layer F.Cu) (net 3))
   (segment (start 94.1 103.78) (end 94.1 102.4) (width 0.4) (layer F.Cu) (net 3))
-  (via (at 93.98 109.3724) (size 0.6) (drill 0.3) (layers F.Cu B.Cu) (net 3))
-  (segment (start 95.9 108.75) (end 95.2776 109.3724) (width 0.6) (layer F.Cu) (net 3))
-  (segment (start 95.2776 109.3724) (end 93.98 109.3724) (width 0.6) (layer F.Cu) (net 3))
-  (segment (start 93.98 108.948136) (end 93.98 109.3724) (width 0.15) (layer F.Cu) (net 3))
-  (segment (start 93.98 108.505) (end 93.98 108.948136) (width 0.15) (layer F.Cu) (net 3))
-  (segment (start 93.675 108.2) (end 93.98 108.505) (width 0.15) (layer F.Cu) (net 3))
-  (segment (start 93.275 108.2) (end 93.675 108.2) (width 0.15) (layer F.Cu) (net 3))
-  (segment (start 93.7728 109.5796) (end 93.98 109.3724) (width 0.6) (layer F.Cu) (net 3))
-  (segment (start 90.92 109.5796) (end 93.7728 109.5796) (width 0.6) (layer F.Cu) (net 3))
   (via (at 93.300006 104.6) (size 0.6) (drill 0.3) (layers F.Cu B.Cu) (net 3))
-  (segment (start 93.300006 108.692406) (end 93.300006 105.024264) (width 0.4) (layer B.Cu) (net 3))
-  (segment (start 93.300006 105.024264) (end 93.300006 104.6) (width 0.4) (layer B.Cu) (net 3))
-  (segment (start 93.98 109.3724) (end 93.300006 108.692406) (width 0.4) (layer B.Cu) (net 3))
   (segment (start 93.3 104.600006) (end 93.300006 104.6) (width 0.6) (layer F.Cu) (net 3))
   (segment (start 93.3 105.35) (end 93.3 104.600006) (width 0.6) (layer F.Cu) (net 3))
@@
   (segment (start 94.1 103.800006) (end 93.300006 104.6) (width 0.4) (layer F.Cu) (net 3))
   (segment (start 94.1 103.78) (end 94.1 103.800006) (width 0.4) (layer F.Cu) (net 3))
+  (via (at 93.98 109) (size 0.6) (drill 0.3) (layers F.Cu B.Cu) (net 3))
+  (segment (start 93.300006 108.320006) (end 93.680001 108.700001) (width 0.4) (layer B.Cu) (net 3))
+  (segment (start 94.279999 109.299999) (end 93.98 109) (width 0.6) (layer F.Cu) (net 3))
+  (segment (start 93.98 108.505) (end 93.98 108.575736) (width 0.15) (layer F.Cu) (net 3))
+  (segment (start 93.98 108.575736) (end 93.98 109) (width 0.15) (layer F.Cu) (net 3))
+  (segment (start 93.675 108.2) (end 93.98 108.505) (width 0.15) (layer F.Cu) (net 3))
+  (segment (start 93.300006 104.6) (end 93.300006 108.320006) (width 0.4) (layer B.Cu) (net 3))
+  (segment (start 93.275 108.2) (end 93.675 108.2) (width 0.15) (layer F.Cu) (net 3))
+  (segment (start 95.35 109.3) (end 94.279999 109.299999) (width 0.6) (layer F.Cu) (net 3))
+  (segment (start 95.9 108.75) (end 95.35 109.3) (width 0.6) (layer F.Cu) (net 3))
+  (segment (start 93.680001 108.700001) (end 93.98 109) (width 0.4) (layer B.Cu) (net 3))
+  (segment (start 94.279999 109.320001) (end 94.279999 109.299999) (width 0.4) (layer F.Cu) (net 3))
+  (segment (start 93.8 109.8) (end 94.279999 109.320001) (width 0.4) (layer F.Cu) (net 3))
   (segment (start 92.6146 107.0396) (end 93.275 107.7) (width 0.15) (layer F.Cu) (net 4))
   (segment (start 90.92 107.0396) (end 92.6146 107.0396) (width 0.15) (layer F.Cu) (net 4))
@@
   (segment (start 105 102) (end 105.399999 102.399999) (width 0.15) (layer B.Cu) (net 33))
   (segment (start 105.9 106.5) (end 105.1 105.7) (width 0.15) (layer F.Cu) (net 33))
+  (segment (start 91.1404 109.8) (end 90.92 109.5796) (width 0.4) (layer F.Cu) (net 34))
+  (segment (start 93 109.8) (end 91.1404 109.8) (width 0.4) (layer F.Cu) (net 34))
   (zone (net 2) (net_name GND) (layer F.Cu) (hatch edge 0.508)
     (connect_pads (clearance 0.15))
